File: Circuit/Circuit.kicad_sch (KiCad schematic)
At the start: 35 parts, among them J1 USB_B_Micro, Q1 SS8050-G, Q2 SS8050-G, SW1 SW_SPST, SW2 SW_SPST, U1 CP2102N-Axx-xQFN28, U1 NodeMCU1.0(ESP-12E), U2 AMS1117-3.3, U2 DS18B20, U3 ESP32-WROVER-I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

Commit message: latest
Parts:
- removed D1: 19-C47/RSGHBHC-5V01/2T, 19-C47_RSGHBHC-5V01_2T:LED_19-C47_RSGHBHC-5V01_2T, symbol 19-C47_RSGHBHC-5V01_2T:19-C47/RSGHBHC-5V01/2T
- removed U1: NodeMCU1.0(ESP-12E), 113990105:SEEED_113990105, symbol ESP8266:NodeMCU1.0(ESP-12E)
Changed lines of the file:
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@@
-    (stroke (width 0) (type default) (color 0 0 0 0))
-  )
-  (wire (pts (xy 248.92 63.5) (xy 248.92 68.58))
     (stroke (width 0) (type default) (color 0 0 0 0))
   )
@@
     (stroke (width 0) (type default) (color 0 0 0 0))
   )
-  (wire (pts (xy 240.03 63.5) (xy 248.92 63.5))
-    (stroke (width 0) (type default) (color 0 0 0 0))
-  )
   (wire (pts (xy 26.67 163.83) (xy 26.67 173.99))
     (stroke (width 0) (type default) (color 0 0 0 0))
@@
     (stroke (width 0) (type default) (color 0 0 0 0))
   )
-  (wire (pts (xy 193.04 66.04) (xy 193.04 64.77))
-    (stroke (width 0) (type default) (color 0 0 0 0))
-  )
   (wire (pts (xy 275.59 101.6) (xy 264.16 101.6))
     (stroke (width 0) (type default) (color 0 0 0 0))
@@
     (stroke (width 0) (type default) (color 0 0 0 0))
   )
-  (wire (pts (xy 199.39 66.04) (xy 193.04 66.04))
-    (stroke (width 0) (type default) (color 0 0 0 0))
-  )
   (wire (pts (xy 22.86 73.66) (xy 22.86 74.93))
     (stroke (width 0) (type default) (color 0 0 0 0))
@@
   )
   (label "TXD0" (at 166.37 133.35 0)
+    (effects (font (size 1.27 1.27)) (justify left bottom))
+  )
+  (label "IO12" (at 240.03 49.53 0)
     (effects (font (size 1.27 1.27)) (justify left bottom))
   )
@@
     (pin "1")
   )
-  (symbol (lib_id "19-C47_RSGHBHC-5V01_2T:19-C47{slash}RSGHBHC-5V01{slash}2T") (at 168.91 30.48 0) (unit 1)
-    (in_bom yes) (on_board yes) (fields_autoplaced)
-    (property "Reference" "D1" (id 0) (at 168.91 17.78 0))
-    (property "Value" "19-C47/RSGHBHC-5V01/2T" (id 1) (at 168.91 20.32 0))
-    (property "Footprint" "19-C47_RSGHBHC-5V01_2T:LED_19-C47_RSGHBHC-5V01_2T" (id 2) (at 168.91 30.48 0)
-      (effects (font (size 1.27 1.27)) (justify bottom) hide)
-    )
-    (property "Datasheet" "" (id 3) (at 168.91 30.48 0)
-      (effects (font (size 1.27 1.27)) hide)
-    )
-    (property "STANDARD" "Manufacturer Recommendations" (id 4) (at 168.91 30.48 0)
-      (effects (font (size 1.27 1.27)) (justify bottom) hide)
-    )
-    (property "MAXIMUM_PACKAGE_HEIGHT" "0.65 mm" (id 5) (at 168.91 30.48 0)
-      (effects (font (size 1.27 1.27)) (justify bottom) hide)
-    )
-    (property "MANUFACTURER" "Everlight Electronics Co Ltd" (id 6) (at 168.91 30.48 0)
-      (effects (font (size 1.27 1.27)) (justify bottom) hide)
-    )
-    (property "PARTREV" "5" (id 7) (at 168.91 30.48 0)
-      (effects (font (size 1.27 1.27)) (justify bottom) hide)
-    )
-    (pin "1")
-    (pin "2")
-    (pin "3")
-    (pin "4")
-  )
   (symbol (lib_id "power:GND") (at 146.05 90.17 0) (unit 1)
     (in_bom yes) (on_board yes) (fields_autoplaced)
@@
     (pin "1")
   )
-  (symbol (lib_id "power:+5V") (at 193.04 64.77 0) (unit 1)
-    (in_bom yes) (on_board yes) (fields_autoplaced)
-    (property "Reference" "#PWR0103" (id 0) (at 193.04 68.58 0)
-      (effects (font (size 1.27 1.27)) hide)
-    )
-    (property "Value" "+5V" (id 1) (at 193.04 59.69 0))
-    (property "Footprint" "" (id 2) (at 193.04 64.77 0)
-      (effects (font (size 1.27 1.27)) hide)
-    )
-    (property "Datasheet" "" (id 3) (at 193.04 64.77 0)
-      (effects (font (size 1.27 1.27)) hide)
-    )
-    (pin "1")
-  )
   (symbol (lib_id "Device:Battery") (at 74.93 80.01 0) (unit 1)
     (in_bom yes) (on_board yes) (fields_autoplaced)
@@
     )
     (property "Datasheet" "" (id 3) (at 264.16 109.22 0)
-      (effects (font (size 1.27 1.27)) hide)
-    )
-    (pin "1")
-  )
-  (symbol (lib_id "power:GND") (at 248.92 68.58 0) (unit 1)
-    (in_bom yes) (on_board yes) (fields_autoplaced)
-    (property "Reference" "#PWR0102" (id 0) (at 248.92 74.93 0)
-      (effects (font (size 1.27 1.27)) hide)
-    )
-    (property "Value" "GND" (id 1) (at 248.92 73.66 0))
-    (property "Footprint" "" (id 2) (at 248.92 68.58 0)
-      (effects (font (size 1.27 1.27)) hide)
-    )
-    (property "Datasheet" "" (id 3) (at 248.92 68.58 0)
       (effects (font (size 1.27 1.27)) hide)
     )
@@
     (pin "2")
   )
-  (symbol (lib_id "ESP8266:NodeMCU1.0(ESP-12E)") (at 219.71 48.26 0) (unit 1)
-    (in_bom yes) (on_board yes) (fields_autoplaced)
-    (property "Reference" "U1" (id 0) (at 219.71 20.32 0)
-      (effects (font (size 1.524 1.524)))
-    )
-    (property "Value" "NodeMCU1.0(ESP-12E)" (id 1) (at 219.71 24.13 0)
-      (effects (font (size 1.524 1.524)))
-    )
-    (property "Footprint" "113990105:SEEED_113990105" (id 2) (at 204.47 69.85 0)
-      (effects (font (size 1.524 1.524)) hide)
-    )
-    (property "Datasheet" "" (id 3) (at 204.47 69.85 0)
-      (effects (font (size 1.524 1.524)))
-    )
-    (pin "1")
-    (pin "10")
-    (pin "11")
-    (pin "12")
-    (pin "13")
-    (pin "14")
-    (pin "15")
-    (pin "16")
-    (pin "17")
-    (pin "18")
-    (pin "19")
-    (pin "2")
-    (pin "20")
-    (pin "21")
-    (pin "22")
-    (pin "23")
-    (pin "24")
-    (pin "25")
-    (pin "26")
-    (pin "27")
-    (pin "28")
-    (pin "29")
-    (pin "3")
-    (pin "30")
-    (pin "4")
-    (pin "5")
-    (pin "6")
-    (pin "7")
-    (pin "8")
-    (pin "9")
-  )
   (symbol (lib_id "Device:R") (at 82.55 149.86 0) (unit 1)
     (in_bom yes) (on_board yes) (fields_autoplaced)
@@
       (reference "#PWR0101") (unit 1) (value "GND") (footprint "")
     )
-    (path "/b1a48aae-fe3d-4e58-a9bb-a4bc259c2405"
-      (reference "#PWR0102") (unit 1) (value "GND") (footprint "")
-    )
-    (path "/5755092d-811f-41d4-8765-e442e851774e"
-      (reference "#PWR0103") (unit 1) (value "+5V") (footprint "")
-    )
     (path "/4989aa8e-8d52-4570-966f-eaf98ab832ad"
       (reference "#PWR0104") (unit 1) (value "+5V") (footprint "")
@@
       (reference "C21") (unit 1) (value "100nF") (footprint "")
     )
-    (path "/19d8081e-a449-4264-ae91-25936a7e5695"
-      (reference "D1") (unit 1) (value "19-C47/RSGHBHC-5V01/2T") (footprint "19-C47_RSGHBHC-5V01_2T:LED_19-C47_RSGHBHC-5V01_2T")
-    )
     (path "/f461b4d0-68a5-4076-bd81-e8c72103848d"
       (reference "D1") (unit 1) (value "RED LED") (footprint "")
@@
       (reference "U1") (unit 1) (value "CP2102N-Axx-xQFN28") (footprint "Package_DFN_QFN:QFN-28-1EP_5x5mm_P0.5mm_EP3.35x3.35mm")
     )
-    (path "/daa0a5c0-ca0c-4237-b6ad-aedfd7e58881"
-      (reference "U1") (unit 1) (value "NodeMCU1.0(ESP-12E)") (footprint "113990105:SEEED_113990105")
-    )
     (path "/0ffc6c94-1bca-45d0-a1ba-68cb46785ece"

Commit message: updated sch
Parts:
- removed U2: DS18B20, Package_TO_SOT_THT:TO-92_Inline, symbol Sensor_Temperature:DS18B20
- added J2: Heater, Connector_Molex:Molex_KK-254_AE-6410-02A_1x02_P2.54mm_Vertical, symbol Connector_Generic:Conn_01x02
- added J3: Temp Sensor, Connector_Molex:Molex_KK-254_AE-6410-03A_1x03_P2.54mm_Vertical, symbol Connector_Generic:Conn_01x03
- added J4: RGB LED, Connector_Molex:Molex_KK-254_AE-6410-04A_1x04_P2.54mm_Vertical, symbol Connector_Generic:Conn_01x04
- added PS1: MEE1S0305SC, Converter_DCDC:Converter_DCDC_Murata_MEE1SxxxxSC_THT, symbol Converter_DCDC:MEE1S0305SC
- added Q3: DMN2058U, Package_TO_SOT_SMD:SOT-23, symbol Transistor_FET:DMN2058U
- added R6: 100, Resistor_SMD:R_0805_2012Metric_Pad1.20x1.40mm_HandSolder, symbol Device:R
- added R7: 10k, Resistor_SMD:R_0805_2012Metric_Pad1.20x1.40mm_HandSolder, symbol Device:R
- C1: footprint (none) -> Capacitor_SMD:C_0805_2012Metric_Pad1.18x1.45mm_HandSolder
- C2: renamed from C3; footprint (none) -> Capacitor_SMD:C_0805_2012Metric_Pad1.18x1.45mm_HandSolder
- C3: renamed from C15; footprint (none) -> Capacitor_SMD:C_0805_2012Metric_Pad1.18x1.45mm_HandSolder
- C4: renamed from C19; footprint (none) -> Capacitor_SMD:C_0805_2012Metric_Pad1.18x1.45mm_HandSolder
- C5: renamed from C20; footprint (none) -> Capacitor_SMD:C_0805_2012Metric_Pad1.18x1.45mm_HandSolder
- C6: renamed from C14; footprint (none) -> Capacitor_SMD:C_0805_2012Metric_Pad1.18x1.45mm_HandSolder
- C7, C8: renamed from C21; footprint (none) -> Capacitor_SMD:C_0805_2012Metric_Pad1.18x1.45mm_HandSolder
- D2: renamed from D6; footprint TVS_LESD5D5.0CT1G -> LESD5D5:TVS_LESD5D5.0CT1G
- D3: renamed from D4; footprint TVS_LESD5D5.0CT1G -> LESD5D5:TVS_LESD5D5.0CT1G
- D4: renamed from D5; footprint TVS_LESD5D5.0CT1G -> LESD5D5:TVS_LESD5D5.0CT1G
- Q1, Q2: footprint TRANS_SS8050-G -> SS8050-G:TRANS_SS8050-G
- R1: renamed from R2; footprint (none) -> Resistor_SMD:R_0805_2012Metric_Pad1.20x1.40mm_HandSolder
- R11: footprint (none) -> Resistor_SMD:R_0805_2012Metric_Pad1.20x1.40mm_HandSolder
- R2: renamed from R21; footprint (none) -> Resistor_SMD:R_0805_2012Metric_Pad1.20x1.40mm_HandSolder
- R3: renamed from R22; footprint (none) -> Resistor_SMD:R_0805_2012Metric_Pad1.20x1.40mm_HandSolder
- R4: renamed from R25; footprint (none) -> Resistor_SMD:R_0805_2012Metric_Pad1.20x1.40mm_HandSolder
- R5: renamed from R26; footprint (none) -> Resistor_SMD:R_0805_2012Metric_Pad1.20x1.40mm_HandSolder
- R8: renamed from R23; footprint (none) -> Resistor_SMD:R_0805_2012Metric_Pad1.20x1.40mm_HandSolder
- U1: renamed from U3; footprint XCVR_ESP32-WROVER-I -> ESP32-WROVER-I:XCVR_ESP32-WROVER-I
- renumbered R18 to R10, R1 to R12, R17 to R9, U1 to U2, U4 to U3, U2 to U4
Connections:
- net +5V: now also J2.1 (Pin_1), J3.3 (Pin_3)
- net GND: now also J3.1 (Pin_1), J4.1 (Pin_1), J4.2 (Pin_2), J4.4 (Pin_4), PS1.1 (-Vin), PS1.3 (-Vout), Q3.2 (S), R7.2
- net IO12: now also R12.1, J3.2 (Pin_2)
- net IO18: now also J4.3 (Pin_3)
- net IO23: now also PS1.2 (+Vin)
- new net: PS1.4 (+Vout), R6.1
- new net: Q3.1 (G), R6.2, R7.1
- new net: J2.2 (Pin_2), Q3.3 (D)
Other:
- note added: "Control Module"
- note added: "Heating Module"
- note added: "LED Module"
- note added: "Sensor Module"
- moved on the sheet: C6, C7, C8, R11, R12, SW2, U1

Commit message: Update PCB
Parts:
- removed D1: RED LED, symbol Device:LED
- added D1, D5: LTST-C171KRKT, LTST-C171KRKT:DIOC200X125X110, symbol LTST-C171KRKT:LTST-C171KRKT
- added J5: Power Supply, Connector_Molex:Molex_KK-254_AE-6410-02A_1x02_P2.54mm_Vertical, symbol Connector_Generic:Conn_01x02
- added R13: 2K, Resistor_SMD:R_0805_2012Metric_Pad1.20x1.40mm_HandSolder, symbol Device:R
- added R14: 5.1K, Resistor_SMD:R_0805_2012Metric_Pad1.20x1.40mm_HandSolder, symbol Device:R
- R10, R9: footprint (none) -> Resistor_SMD:R_0805_2012Metric_Pad1.20x1.40mm_HandSolder
- SW1, SW2: footprint (none) -> Button_Switch_SMD:SW_Push_1P1T_NO_CK_KSC6xxJ
- U3: footprint (none) -> TP4056-18650:TP4056-18650
Connections:
- net +5C is gone; now on net +5V: R4.1
- net +3.3V: now also J3.3 (Pin_3), R12.2, R13.1, R14.1
- net +5V: now also J5.1 (Pin_1); no longer J3.3 (Pin_3), R12.2
- net GND: now also D1.-, D5.-, J5.2 (Pin_2)
- net USB_DP: now also U2.4 (D+)
- net at R1.2: now also D1.+
- net at U2.9 (~{RST}): now also R13.2
- new net: D5.+, R14.2
- no-connect marks 7 -> 18
Other:
- moved on the sheet: C3, C6, R11, SW1, SW2
