File: Circuit/Circuit.kicad_pcb (KiCad board)
At the start: 2 copper layers, 41 parts, among them J1 USB_B_Micro, J2 Heater, J3 Temp Sensor, J4 RGB LED, J5 Power Supply, Q1 SS8050-G, Q2 SS8050-G, Q3 DMN2058U, SW1 SW_SPST, SW2 SW_SPST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

Commit message: update log
Routing:
- net GND: track 17.7 -> 19.5 mm, vias 50 -> 51
